File: dcmotor_controller.sch (EAGLE design)
At the start: 69 parts, among them IC1 L298, IC2 L298, IC3 AS5040, IC4 7805DT, IC5 SN74LVCR162245A, Q1 8MHz, U1 STM32F051C8T6

Commit message: Add files via upload
Parts:
- removed C17, C18: 100n, rcl:C-EU025-024X044
- removed C19: 1u, rcl:C-EU025-024X044
- removed C21, C22: 20p, rcl:C-EU025-024X044
- removed IC4: 7805DT, linear:7805DT
- removed Q1: 8MHz, crystal:CSM-7X-DU
- removed U1: STM32F051C8T6, untitled:STM32F051C8T6
- added C25: 4u7, rcl:C-EU025-024X044
- added C26, C27, C28, C30: 100n, rcl:C-EU025-024X044
- added C29: 1u, rcl:C-EU025-024X044
- added C31, C32: 20p, rcl:C-EU025-024X044
- added D18: SMBJ5.0A-TR, diode:SUPPRESSOR-SMBJ
- added F1: SL125-33, polyfuse-smd_10:2920L050
- added LED, POWER_CON: (no value), con-ptr500:AK500/2
- added Q2: 8MHz, crystal:CSM-7X-DU
- added R19, R20: 10k 1%, resistor:R-EU_M0805
- added R45: 10k, resistor:R-EU_M0805
- added R46: 2k2, resistor:R-EU_M0805
- added R48: 100k, resistor:R-EU_M0805
- added R49: 100, resistor:R-EU_M0805
- added SV2, SV3, SV4, SV5: (no value), con-ml:ML10L
- added SV6: (no value), con-lsta:FE20-2
- added T1: (no value), we-transistor:MOSFET-P-SOT23
- added T14: BSS306N, we-transistor:MOSFET-N-SOT23
- added U$2: LM2596_CONVERTER, Voltage Converter:LM2596_CONVERTER
- added U$3: BCM857BS, BCM857BS:BCM857BS
- added U2: STM32F10XRXT6, stm32:STM32F10XRXT6
- added X3: (no value), con-phoenix-254:MPT2
- C10: value 10u -> 100u; device rcl:CPOL-EU140CLH-0810 -> resistor:CPOL-EU153CLV-0807; LINK (none) -> http://www.tme.eu/pl/details/sc1e107m0806bvr/kondensatory-e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
- C15: value 4u7 -> 100n; device rcl:C-EU025-024X044 -> resistor:C-EUC0805
- C16: device rcl:C-EU025-024X044 -> resistor:C-EUC0805
- C20: value 100n -> 47u; device rcl:C-EU025-024X044 -> resistor:C-EUC0805; LINK (none) -> http://www.tme.eu/pl/details/cl21a476mqynnng/kondensatory-m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
- C9: value 100u -> 4u7; device rcl:CPOL-EU140CLH-0810 -> resistor:C-EUC0805
Connections:
- removed net N$3: C9.+, IC4.VI
- new net +3V3: SV6.1, SV6.17
- new net +5V: C16.1, D18.C, SV6.2, SV6.4, T1.S, U$3G2.E
- new net MISO: U2PORTB_L.PB4
- new net MOSI: U2PORTB_L.PB5
- new net N$11: C30.1
- new net N$12: C29.1
- new net N$14: U2PORTB_H.PB10
- new net N$15: U2PORTB_H.PB11
- new net N$16: U2AN_POWER.VBAT
- new net N$17: R20.2, T1.G, U$3G2.C
- new net N$18: R19.2, U$3G1.B, U$3G1.C, U$3G2.B
- new net N$21: R48.2, R49.1, T14.G
- new net N$24: LED-1.KL, T14.D
- new net OSC_IN: C31.2, Q2.2, U2PORTD/OSC.PD0/OSC<=
- new net OSC_OUT: C32.2, Q2.1, U2PORTD/OSC.PD1/OSC=>
- new net SCK: U2PORTB_L.PB3
- net A_LSB_U: now also SV2.2, SV3.2, SV4.2, SV5.2
- net BAT_MEAS: now also C20.1, R45.1, R46.2, U2PORTA_L.PA4; no longer U1A.PA4
- net BOOTO: now also U2RESET.BOOT0; no longer U1B.BOOT0
- net B_DIR_V: now also SV2.3, SV3.3, SV4.3, SV5.3
- net CLK: now also SV2.6, SV3.6, SV4.6, SV5.6
- net CSN: now also SV2.5, SV3.5, SV4.5, SV5.5
- net D0: now also SV2.7, SV3.7, SV4.7, SV5.7
- net EN1_UC: now also U2PORTA_L.PA6; no longer U1A.PA6
- net EN2_UC: now also U2PORTA_L.PA7; no longer U1A.PA7
- net EN3_UC: now also U2PORTB_L.PB0; no longer U1A.PB0
- net EN4_UC: now also U2PORTB_L.PB1; no longer U1A.PB1
- net GND: now also C25.2, C26.2, C27.2, C28.2, C29.2, C30.2, C31.1, C32.1, C9.2, D18.A, POWER_CON-1.KL, R19.1, R20.1, R46.1, R48.1, SV2.10, SV3.10, SV4.10, SV5.10, SV6.14, SV6.20, SV6.25, SV6.30, SV6.34, SV6.39, SV6.6, SV6.9, T14.S, U$2.GND0, U$2.GND2, U2AN_POWER.VSSA, U2POWER.VSS_1, U2POWER.VSS_2, U2POWER.VSS_3, U2POWER.VSS_4, X3-2.1; no longer C17.2, C18.2, C19.2, C21.1, C22.1, C9.-, IC4.GND, U1A.VSS, U1A.VSSA, U1B.VSS
- net IN11_UC: now also U2PORTC_L.PC0; no longer U1B.PB8
- net IN12_UC: now also U2PORTC_L.PC1; no longer U1B.PB9
- net IN21_UC: now also U2PORTC_L.PC2; no longer U1A.PB10
- net IN22_UC: now also U2PORTC_L.PC3; no longer U1A.PB11
- net IN31_UC: now also U2PORTC_L.PC4; no longer U1B.PB12
- net IN32_UC: now also U2PORTC_L.PC5; no longer U1B.PB13
- net IN41_UC: now also U2PORTC_L.PC6; no longer U1B.PB14
- net IN42_UC: now also U2PORTC_L.PC7; no longer U1B.PB15
- net INDEX_W: now also SV2.4, SV3.4, SV4.4, SV5.4
- net LED: now also R49.2, U2PORTA_L.PA5; no longer U1A.PA5
- net N$5: now also F1.2, U$2.+5V; no longer C21.2, Q1.2, U1A.PF0/OSC_IN
- net N$6: now also C15.1, F1.1, T1.D, U$3G1.E; no longer C22.2, Q1.1, U1A.PF1/OSC_OUT
- net NRST: now also SV6.12, U2RESET.NRST; no longer U1A.NRST
- net PWM: now also SV2.9, SV3.9, SV4.9, SV5.9
- net PWM_F: now also SV2.8, SV3.8, SV4.8, SV5.8
- net RPI_CLK: now also SV6.23; no longer U1B.PB3
- net RPI_MISO: now also SV6.21; no longer U1B.PB4
- net RPI_MOSI: now also SV6.19; no longer U1B.PB5
- net RPI_RXD: now also SV6.10, U2PORTB_L.PB6; no longer U1B.PB6
- net RPI_TXD: now also SV6.8, U2PORTB_L.PB7; no longer U1B.PB7
- net SCL: now also SV6.5; no longer U1B.PF6
- net SDA: now also SV6.3; no longer U1B.PF7
- net SEN1: now also U2PORTA_L.PA0; no longer U1A.PA0
- net SEN2: now also U2PORTA_L.PA1; no longer U1A.PA1
- net SEN3: now also U2PORTA_L.PA2; no longer U1A.PA2
- net SEN4: now also U2PORTA_L.PA3; no longer U1A.PA3
- net SPI1_NSS: now also SV6.15, SV6.24, U2PORTA_H.PA15; no longer U1B.PA15
- net SWCLK: now also SV6.22, U2PORTA_H.PA14; no longer U1B.PA14
- net SWDIO: now also SV6.18, U2PORTA_H.PA13; no longer U1B.PA13
- net VCC: now also C9.1, LED-2.KL, POWER_CON-2.KL, R45.2, SV2.1, SV3.1, SV4.1, SV5.1, U$2.VIN+, X3-1.1; no longer IC4.VO
- net VDD: now also C25.1, C26.1, C27.1, C28.1, U2AN_POWER.VDDA, U2POWER.VDD_1, U2POWER.VDD_2, U2POWER.VDD_3, U2POWER.VDD_4; no longer C15.1, C16.1, C17.1, C18.1, C19.1, C20.1, U1A.VDD, U1A.VDDA, U1B.VDD
Other:
- note removed: "MICROCONTROLER STM32F05"
- moved on the sheet: C10, C15, C16, C20, C5, C6, C7, C8, IC3, LED1, R1, R10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
