File: dcmotor_controller.sch (EAGLE design)
At the start: 87 parts, among them IC1 L298, IC2 L298, Q1 MOSFET-PCHANNEL_SOT23-3, Q2 8MHz, T1 BC857BS, T14 BSS306N, U1 SN74LVC4245APWR, U2 STM32F10XRXT6, U3 SN74LVC4245APWR, U4 MCP1825S-3302E/DB

Commit message: renumber parts, small changes in layout
Parts:
- removed C30: 100n, rcl:C-EUC0805
- removed C31, C32: 20p, rcl:C-EUC0805
- removed LED: (no value), con-ptr500:AK500/2
- removed R19: 1.2k, 0.5W, rcl:R-EU_R2010
- removed R20: 0R25, rcl:R-EU_R2512
- removed R45, R62: 10k, resistor:R-EU_M0805
- removed R46: 2k2, resistor:R-EU_M0805
- removed SV6: (no value), con-lsta:FE20-2
- removed T14: BSS306N, we-transistor:MOSFET-N-SOT23
- removed U$1: DC-DC-STEP-DOWN-LM2596, lm2596:DC-DC-STEP-DOWN-LM2596
- added C22: 10u, resistor:CPOL-EU153CLV-0807
- added C23: 100n, resistor:C-EUC0805
- added C24: (no value), rcl:C-EUC0805
- added R17, R18: 10k 1%, resistor:R-EU_M0805
- added R2: 0R25, rcl:R-EU_R2512
- added R6: 10k, resistor:R-EU_M0805
- added R9: (no value), rcl:R-EU_R0805
- added SV1: (no value), con-ml:ML10L
- added T2: BC857BS, NXP_60_26022015:BC857BS
- added U5: MCP1825S-3302E/DB, MCP1825S-3302E_DB:MCP1825S-3302E/DB
- added X5: (no value), con-phoenix-254:MPT2
- C10: value 100u -> 100n; device resistor:CPOL-EU153CLV-0807 -> resistor:C-EUC0805; LINK http://www.tme.eu/pl/details/sc1e107m0806bvr/kondensatory-e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 -> (none)
- C13: value 100n -> 4u7; device resistor:C-EUC0805 -> rcl:C-EUC0805
- C14, C3: device resistor:C-EUC0805 -> rcl:C-EUC0805
- C15: value 100n -> 20p; device resistor:C-EUC0805 -> rcl:C-EUC0805; LINK http://www.tme.eu/pl/details/cl21a476mqynnng/kondensatory-m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 -> (none)
- C16: value 100n -> 20p; device resistor:C-EUC0805 -> rcl:C-EUC0805
- C17: device resistor:C-EUC0805 -> rcl:C-EUC0805; LINK http://www.tme.eu/pl/details/cl21a476mqynnng/kondensatory-m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 -> (none)
- C18: value 10u -> 100n; device resistor:CPOL-EU153CLV-0807 -> rcl:C-EUC0805; LINK http://www.tme.eu/pl/details/sc1e107m0806bvr/kondensatory-e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 -> (none)
- C19: value 10u -> 1u; device resistor:CPOL-EU153CLV-0807 -> rcl:C-EUC0805; LINK http://www.tme.eu/pl/details/sc1e107m0806bvr/kondensatory-e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 -> (none)
- C2, C25: device rcl:C-EUC0805 -> resistor:C-EUC0805
- C20: value 47u -> 100n; device resistor:C-EUC0805 -> rcl:C-EUC0805; LINK http://www.tme.eu/pl/details/cl21a476mqynnng/kondensatory-m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 -> (none)
- C21: value 100n -> 47u; LINK (none) -> http://www.tme.eu/pl/details/cl21a476mqynnng/kondensatory-m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
- C26: device rcl:C-EUC0805 -> resistor:C-EUC0805; LINK (none) -> http://www.tme.eu/pl/details/cl21a476mqynnng/kondensatory-m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
- C27: value 100n -> 10u; device rcl:C-EUC0805 -> resistor:CPOL-EU153CLV-0807; LINK (none) -> http://www.tme.eu/pl/details/sc1e107m0806bvr/kondensatory-e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
- C28: value 100n -> 100u; device rcl:C-EUC0805 -> resistor:CPOL-EU153CLV-0807; LINK (none) -> http://www.tme.eu/pl/details/sc1e107m0806bvr/kondensatory-e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
- C29: value 1u -> 100n; device rcl:C-EUC0805 -> resistor:C-EUC0805
- C5: value (none) -> 100n; device rcl:C-EUC0805 -> resistor:C-EUC0805
- C9: value 4u7 -> 100n
- Q1: value MOSFET-PCHANNEL_SOT23-3 -> 8MHz; device Simplex-DiscreteSemi:MOSFET-PCHANNEL_SOT23-3 -> crystal:CSM-7X-DU
- Q2: value 8MHz -> MOSFET-PCHANNEL_SOT23-3; device crystal:CSM-7X-DU -> Simplex-DiscreteSemi:MOSFET-PCHANNEL_SOT23-3
- R1: value 10k -> 0R25; device resistor:R-EU_M0805 -> rcl:R-EU_R2512; LINK (none) -> http://www.tme.eu/pl/details/cs2512-0r25-1%25-hp/rezystory-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
- R12: value 10k -> 1.2k, 0.5W; device rcl:R-EU_R0805 -> rcl:R-EU_R2010
- R13: device rcl:R-EU_R0805 -> resistor:R-EU_M0805
- R14: value (none) -> 2k2; device rcl:R-EU_R0805 -> resistor:R-EU_M0805
- R5: value 0R25 -> 10k; device rcl:R-EU_R2512 -> resistor:R-EU_M0805; LINK http://www.tme.eu/pl/details/cs2512-0r25-1%25-hp/rezystory-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 -> (none)
- R7, R8: value 10k 1% -> 10k; device resistor:R-EU_M0805 -> rcl:R-EU_R0805
- SV5: device con-ml:ML10L -> con-lsta:FE20-2
- T1: value BC857BS -> BSS306N; device NXP_60_26022015:BC857BS -> we-transistor:MOSFET-N-SOT23
- U1: value SN74LVC4245APWR -> STM32F10XRXT6; device Texas Instruments_By_element14_Batch_1:SN74LVC4245APWR -> stm32:STM32F10XRXT6
- U2: value STM32F10XRXT6 -> SN74LVC4245APWR; device stm32:STM32F10XRXT6 -> Texas Instruments_By_element14_Batch_1:SN74LVC4245APWR
- U4: value MCP1825S-3302E/DB -> DC-DC-STEP-DOWN-LM2596; device MCP1825S-3302E_DB:MCP1825S-3302E/DB -> lm2596:DC-DC-STEP-DOWN-LM2596
- X3: device con-phoenix-254:MPT2 -> con-ptr500:AK500/2
- renumbered D19 to D1, F2 to F1, LED2 to LED1, PWR to X4, R48 to R16, R49 to R15
Connections:
- net 24V: now also C25.1, C28.+, C3.1, D11.C, D13.C, D15.C, D9.C, R12.1, R13.2, U4.IN+, X3-2.KL, X5-1.1; no longer C10.+, C2.1, C9.1, D2.C, D4.C, D6.C, D8.C, LED-2.KL, R19.1, R45.2, U$1.IN+, X3-1.1
- net 3V3: now also C10.1, C13.1, C18.1, C19.1, C20.1, C27.+, C9.1, R7.2, R9.2, SV1.1, U1AN_POWER.VDDA, U1POWER.VDD_1, U1POWER.VDD_2, U1POWER.VDD_3, U1POWER.VDD_4, U2.VCCB_(3.3_V), U2.VCCB_(3.3_V)_2, U5.VOUT; no longer C19.+, C25.1, C27.1, C28.1, C29.1, C30.1, C7.1, R12.2, R14.2, SV5.1, U1.VCCB_(3.3_V), U1.VCCB_(3.3_V)_2, U2AN_POWER.VDDA, U2POWER.VDD_1, U2POWER.VDD_2, U2POWER.VDD_3, U2POWER.VDD_4, U4.VOUT
- net 5V: now also C11.1, C12.1, C2.2, C22.+, C23.1, C29.1, Q2.S, SV5.2, SV5.4, T2-2.E, U2.(5_V)_VCCA, U5.VIN; no longer C15.1, C16.1, C18.+, C3.2, C6.1, C8.1, Q1.S, SV6.2, SV6.4, T1-2.E, U1.(5_V)_VCCA, U4.VIN
- net A_LSB_U1: now also SV1.2, U1PORTA_H.PA8; no longer SV2.2, U2PORTA_H.PA8
- net A_LSB_U2: now also U1PORTA_H.PA9; no longer U2PORTA_H.PA9
- net A_LSB_U3: now also SV2.2, U1PORTA_H.PA10; no longer SV4.2, U2PORTA_H.PA10
- net A_LSB_U4: now also SV4.2, U1PORTA_H.PA11; no longer SV5.2, U2PORTA_H.PA11
- net BAT_MEAS: now also C21.1, R13.1, R14.2, U1PORTA_L.PA4; no longer C20.1, R45.1, R46.2, U2PORTA_L.PA4
- net BOOTO: now also R8.2, U1RESET.BOOT0; no longer R13.2, U2RESET.BOOT0
- net B_DIR_V1: now also SV1.3, U1PORTC_H.PC8; no longer SV2.3, U2PORTC_H.PC8
- net B_DIR_V2: now also U1PORTC_H.PC9; no longer U2PORTC_H.PC9
- net B_DIR_V3: now also SV2.3, U1PORTC_H.PC10; no longer SV4.3, U2PORTC_H.PC10
- net B_DIR_V4: now also SV4.3, U1PORTC_H.PC11; no longer SV5.3, U2PORTC_H.PC11
- net CLK: now also SV1.6, U1PORTB_H.PB8; no longer SV5.6, U2PORTB_H.PB8
- net CSN: now also SV1.5, U1PORTB_H.PB9; no longer SV5.5, U2PORTB_H.PB9
- net D01: now also SV1.7, U1PORTC_H.PC12; no longer SV2.7, U2PORTC_H.PC12
- net D02: now also U1PORTC_H.PC13; no longer U2PORTC_H.PC13
- net D03: now also SV2.7, U1PORTC_H.PC14; no longer SV4.7, U2PORTC_H.PC14
- net D04: now also SV4.7, U1PORTC_H.PC15; no longer SV5.7, U2PORTC_H.PC15
- net EN1_UC: now also U1PORTA_L.PA6, U2.B1; no longer U1.B1, U2PORTA_L.PA6
- net EN2_UC: now also U1PORTA_L.PA7, U2.B2; no longer U1.B2, U2PORTA_L.PA7
- net EN3_UC: now also U1PORTB_L.PB0, U2.B3; no longer U1.B3, U2PORTB_L.PB0
- net EN4_UC: now also U1PORTB_L.PB1, U2.B4; no longer U1.B4, U2PORTB_L.PB1
- net GND: now also C10.2, C11.2, C12.2, C13.2, C15.1, C16.1, C18.2, C19.2, C2.1, C21.2, C22.-, C23.2, C24.2, C27.-, C28.-, C3.2, C5.1, C6.1, C7.1, C8.1, D2.A, D4.A, D6.A, D8.A, R1.1, R14.1, R17.1, R18.1, R2.1, R5.2, R6.2, SV1.10, SV5.14, SV5.20, SV5.25, SV5.30, SV5.34, SV5.39, SV5.6, SV5.9, T1.S, U1AN_POWER.VSSA, U1POWER.VSS_1, U1POWER.VSS_2, U1POWER.VSS_3, U1POWER.VSS_4, U2.GND, U2.GND_2, U2.GND_3, U4.IN-, U4.OUT-, U5.GND_(TAB), U5.GND_(TAB)_2, X5-2.1; no longer C10.-, C11.1, C12.1, C13.1, C15.2, C16.2, C18.-, C19.-, C2.2, C21.1, C27.2, C28.2, C3.1, C30.2, C31.1, C32.1, C5.2, C6.2, C7.2, C8.2, D11.A, D13.A, D15.A, D9.A, R1.2, R13.1, R20.1, R46.1, R5.1, R62.2, R7.1, SV5.10, SV6.14, SV6.20, SV6.25, SV6.30, SV6.34, SV6.39, SV6.6, SV6.9, T14.S, U$1.IN-, U$1.OUT-, U1.GND, U1.GND_2, U1.GND_3, U2AN_POWER.VSSA, U2POWER.VSS_1, U2POWER.VSS_2, U2POWER.VSS_3, U2POWER.VSS_4, U4.GND_(TAB), U4.GND_(TAB)_2, X3-2.1
- net IN11_UC: now also U1PORTC_L.PC0; no longer U2PORTC_L.PC0
- net IN12_UC: now also U1PORTC_L.PC1; no longer U2PORTC_L.PC1
- net IN21_UC: now also U1PORTC_L.PC2; no longer U2PORTC_L.PC2
- net IN22_UC: now also U1PORTC_L.PC3; no longer U2PORTC_L.PC3
- net IN31: now also U2.A5; no longer U1.A5
- net IN31_UC: now also U1PORTC_L.PC4, U2.B5; no longer U1.B5, U2PORTC_L.PC4
- net IN32: now also U2.A6; no longer U1.A6
- net IN32_UC: now also U1PORTC_L.PC5, U2.B6; no longer U1.B6, U2PORTC_L.PC5
- net IN41: now also U2.A7; no longer U1.A7
- net IN41_UC: now also U1PORTC_L.PC6, U2.B7; no longer U1.B7, U2PORTC_L.PC6
- net IN42: now also U2.A8; no longer U1.A8
- net IN42_UC: now also U1PORTC_L.PC7, U2.B8; no longer U1.B8, U2PORTC_L.PC7
- net INDEX_W1: now also SV1.4, U1PORTB_H.PB12; no longer SV2.4, U2PORTB_H.PB12
- net INDEX_W2: now also U1PORTB_H.PB13; no longer U2PORTB_H.PB13
- net INDEX_W3: now also SV2.4, U1PORTB_H.PB14; no longer SV4.4, U2PORTB_H.PB14
- net INDEX_W4: now also SV4.4, U1PORTB_H.PB15; no longer SV5.4, U2PORTB_H.PB15
- net LED: now also U1PORTA_L.PA5; no longer U2PORTA_L.PA5
- net MOT11: now also D2.C; no longer D16.C
- net MOT12: now also D3.A, D4.C; no longer D15.C, D2.A
- net MOT21: now also D5.A, D6.C; no longer D14.C, D3.A
- net MOT22: now also D7.A, D8.C; no longer D13.C, D4.A
- net MOT31: now also D10.C, D9.A; no longer D12.C, D5.A
- net MOT32: now also D11.A, D12.C; no longer D11.C, D6.A
- net MOT41: now also D13.A, D14.C; no longer D10.C, D7.A
- net MOT42: now also D15.A, D16.C; no longer D8.A, D9.C
- net N$1: now also U4.OUT+; no longer U$1.OUT+
- net N$16: now also U1AN_POWER.VBAT; no longer U2AN_POWER.VBAT
- net N$19: now also Q2.G, R18.2, T2-2.C; no longer Q1.G, R8.2, T1-2.C
- net N$20: now also R17.2, T2-1.B, T2-1.C, T2-2.B; no longer R7.2, T1-1.B, T1-1.C, T1-2.B
- net N$21: now also T1.G; no longer T14.G
- net N$24: now also T1.D, X3-1.KL; no longer LED-1.KL, T14.D
- net N$3: now also R12.2; no longer R19.2
- net N$4: now also R5.1, U2.DIR, U2.~OE; no longer R62.1, U1.DIR, U1.~OE
- net N$5: now also R6.1; no longer R1.1
- net N$6: now also C24.1, Q2.D, T2-1.E; no longer C5.1, Q1.D, T1-1.E
- net NRST: now also R7.1, SV5.12, U1RESET.NRST; no longer R12.1, SV6.12, U2RESET.NRST
- net OSC_IN: now also C15.2, Q1.2, U1PORTD/OSC.PD0/OSC<=; no longer C31.2, Q2.2, U2PORTD/OSC.PD0/OSC<=
- net OSC_OUT: now also C16.2, Q1.1, U1PORTD/OSC.PD1/OSC=>; no longer C32.2, Q2.1, U2PORTD/OSC.PD1/OSC=>
- net PWM1: now also SV1.9; no longer SV2.9
- net PWM3: now also SV2.9; no longer SV4.9
- net PWM4: now also SV4.9; no longer SV5.9
- net PWM_F1: now also SV1.8; no longer SV2.8
- net PWM_F3: now also SV2.8; no longer SV4.8
- net PWM_F4: now also SV4.8; no longer SV5.8
- net PWM_SIGNAL1: now also U2.A1; no longer U1.A1
- net PWM_SIGNAL2: now also U2.A2; no longer U1.A2
- net PWM_SIGNAL3: now also U2.A3; no longer U1.A3
- net PWM_SIGNAL4: now also U2.A4; no longer U1.A4
- net RPI_CLK: now also SV5.23, U1PORTB_L.PB3; no longer SV6.23, U2PORTB_L.PB3
- net RPI_MISO: now also SV5.21, U1PORTB_L.PB4; no longer SV6.21, U2PORTB_L.PB4
- net RPI_MOSI: now also SV5.19, U1PORTB_L.PB5; no longer SV6.19, U2PORTB_L.PB5
- net RPI_RXD: now also SV5.10, U1PORTB_L.PB6; no longer SV6.10, U2PORTB_L.PB6
- net RPI_TXD: now also SV5.8, U1PORTB_L.PB7; no longer SV6.8, U2PORTB_L.PB7
- net SCL: now also SV5.5, U1PORTB_H.PB10; no longer SV6.5, U2PORTB_H.PB10
- net SDA: now also SV5.3, U1PORTB_H.PB11; no longer SV6.3, U2PORTB_H.PB11
- net SEN1: now also C5.2, R1.2, U1PORTA_L.PA0; no longer C21.2, R20.2, U2PORTA_L.PA0
- net SEN2: now also C6.2, R2.2, U1PORTA_L.PA1; no longer C11.2, R3.2, U2PORTA_L.PA1
- net SEN3: now also C7.2, R3.2, U1PORTA_L.PA2; no longer C12.2, R4.2, U2PORTA_L.PA2
- net SEN4: now also C8.2, R4.2, U1PORTA_L.PA3; no longer C13.2, R5.2, U2PORTA_L.PA3
- net SPI1_NSS: now also R9.1, SV5.15, SV5.24, U1PORTA_H.PA15; no longer R14.1, SV6.15, SV6.24, U2PORTA_H.PA15
- net SWCLK: now also SV5.22, U1PORTA_H.PA14; no longer SV6.22, U2PORTA_H.PA14
- net SWDIO: now also SV5.18, U1PORTA_H.PA13; no longer SV6.18, U2PORTA_H.PA13
Other:
- moved on the sheet: C11, C12, C13, C14, C15, C16, C17, C2, C20, C21, C25, C26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
